File: ATMEGA328P Datalogger/ATMEGA328P Datalogger.kicad_sch (KiCad schematic)
At the start: 25 parts, among them U1 ATMEGA328P-AU, U2 24LC1025, U3 24LC1025, U4 DS1337S_, Y1 32.768Khz, Y2 16Mhz

Commit message: NET names and seperation has been made
Other:
- note added: "EEPROM"
- note added: "MCU"
- note added: "MOUNTING HOLES"
- note added: "REAL TIME CLOCK"
- moved on the sheet: BT1, C2, C3, C4, C5, D1, D2, R5, R6, R7, U1, Y2
